Commit message: fix(gazebo): port foot bumper plugin ROS1->ROS2 syntax (<ros>/<remapping>/<frame_name>)

File: robot_descriptions/go1_description/urdfs/leg.gazebo.xacro (robot description, xacro)
@@ -3,39 +3,39 @@
     <xacro:macro name="leg_gazebo" params="name load_force_sensors">
         <!-- UNITREE PLUGINS -->
-	    <!-- Foot contact >
-	    <gazebo reference="${name}_lowerleg">
-		    <sensor name="${name}_foot_contact" type="contact">
-		    <update_rate>100</update_rate>
-		    <plugin name="contactPlugin" filename="libunitreeFootContactPlugin.so"/>
-		    <contact>
-		        <collision>${name}_lowerleg_fixed_joint_lump__${name}_foot_collision_1</collision>
-		    </contact>
-		    </sensor>
-	    </gazebo>
-	    <Visualization of Foot contacts. >
-	    <gazebo reference="${name}_foot">
-		    <visual>
-		        <plugin name="drawForcePlugin" filename="libunitreeDrawForcePlugin.so">
-		            <topicName>${name}_foot_contact</topicName>
-		        </plugin>
-		    </visual>
-	    </gazebo-->
-		<gazebo reference="${name}_upperleg">
-			<kp>1000000.0</kp>
-			<kd>100.0</kd>
-			<mu1>1.5</mu1>
-			<mu2>1.5</mu2>
-			<fdir1>1 0 0</fdir1>
-			<maxVel>1.0</maxVel>
-			<minDepth>0.00</minDepth>
-		</gazebo>
-		<gazebo reference="${name}_lowerleg">
-			<kp>1000000.0</kp>
-			<kd>100.0</kd>
-			<mu1>1.0</mu1>
-			<mu2>1.0</mu2>
-			<maxVel>1.0</maxVel>
-			<maxContacts>1</maxContacts>
-		</gazebo>
+            <!-- Foot contact >
+            <gazebo reference="${name}_lowerleg">
+                    <sensor name="${name}_foot_contact" type="contact">
+                    <update_rate>100</update_rate>
+                    <plugin name="contactPlugin" filename="libunitreeFootContactPlugin.so"/>
+                    <contact>
+                        <collision>${name}_lowerleg_fixed_joint_lump__${name}_foot_collision_1</collision>
+                    </contact>
+                    </sensor>
+            </gazebo>
+            <Visualization of Foot contacts. >
+            <gazebo reference="${name}_foot">
+                    <visual>
+                        <plugin name="drawForcePlugin" filename="libunitreeDrawForcePlugin.so">
+                            <topicName>${name}_foot_contact</topicName>
+                        </plugin>
+                    </visual>
+            </gazebo-->
+                <gazebo reference="${name}_upperleg">
+                        <kp>1000000.0</kp>
+                        <kd>100.0</kd>
+                        <mu1>1.5</mu1>
+                        <mu2>1.5</mu2>
+                        <fdir1>1 0 0</fdir1>
+                        <maxVel>1.0</maxVel>
+                        <minDepth>0.00</minDepth>
+                </gazebo>
+                <gazebo reference="${name}_lowerleg">
+                        <kp>1000000.0</kp>
+                        <kd>100.0</kd>
+                        <mu1>1.0</mu1>
+                        <mu2>1.0</mu2>
+                        <maxVel>1.0</maxVel>
+                        <maxContacts>1</maxContacts>
+                </gazebo>
         <gazebo reference="${name}_foot">
             <kp>1000000.0</kp>
@@ -44,21 +44,23 @@
             <mu2>1.0</mu2>
             <maxVel>1.0</maxVel>
-		    <maxContacts>1</maxContacts>
-		            <sensor name="${name}_foot_contact_sensor" type="contact">
-		            <always_on>true</always_on>
-		            <update_rate>1000.0</update_rate>
-		            <contact>
-		                <collision>${name}_lowerleg_fixed_joint_lump__${name}_foot_collision_1</collision>
-		            </contact>
-		            <!-- the sensor readings in terms of force torques are expressed in the lowerleg frame
-		            because gazebo lumps the fake footframe with the real parent link, the normals are in the world frame-->
-		            <plugin name="${name}_foot_bumper" filename="libgazebo_ros_bumper.so">
-		                <bumperTopicName>/go1/${name}_foot_bumper</bumperTopicName>
-		                <!--robotNamespace>solo</robotNamespace-->
-		                <frameName>${name}_foot</frameName>
-		            </plugin>
-		        </sensor>
+                    <maxContacts>1</maxContacts>
+                            <sensor name="${name}_foot_contact_sensor" type="contact">
+                            <always_on>true</always_on>
+                            <update_rate>1000.0</update_rate>
+                            <contact>
+                                <collision>${name}_lowerleg_fixed_joint_lump__${name}_foot_collision_1</collision>
+                            </contact>
+                            <!-- the sensor readings in terms of force torques are expressed in the lowerleg frame
+                            because gazebo lumps the fake footframe with the real parent link, the normals are in the world frame-->
+                            <plugin name="${name}_foot_bumper" filename="libgazebo_ros_bumper.so">
+                                <ros>
+                                    <namespace>/go1</namespace>
+                                    <remapping>bumper_states:=${name}_foot_bumper</remapping>
+                                </ros>
+                                <frame_name>${name}_foot</frame_name>
+                            </plugin>
+                        </sensor>
             <material>Gazebo/Black</material>
         </gazebo>
-	</xacro:macro>
+        </xacro:macro>
 </robot>
