Commit message: fix(go2): convert visual meshes DAE->STL so Gazebo Classic renders the body
Blender 3.4-exported go2 .dae meshes split each link into multiple
material-bound submeshes with non-ASCII material names. Gazebo Classic's
COLLADA loader silently drops these (RViz/assimp renders them fine),
leaving only the primitive foot spheres visible in Gazebo. Converting the
visual meshes to STL (single geometry, no material binding) makes Gazebo
render the full robot. Physics/joints unaffected; color is now default
gray in both viewers.

File: robot_descriptions/go2_description/robots/go2.urdf.xacro (robot description, xacro)
@@ -26,5 +26,5 @@
             <origin rpy="0 0 0" xyz="0 0 0"/>
             <geometry>
-                <mesh filename="package://go2_description/meshes/trunk.dae" scale="1 1 1"/>
+                <mesh filename="package://go2_description/meshes/trunk.stl" scale="1 1 1"/>
             </geometry>
             <!-- <material name="orange"/> -->

File: robot_descriptions/go2_description/urdfs/leg.xacro (robot description, xacro)
@@ -44,5 +44,5 @@
                 </xacro:if>
                 <geometry>
-                    <mesh filename="package://go2_description/meshes/hip.dae" scale="1 1 1"/>
+                    <mesh filename="package://go2_description/meshes/hip.stl" scale="1 1 1"/>
                 </geometry>
                 <!-- <material name="orange"/> -->
@@ -76,8 +76,8 @@
                 <geometry>
                     <xacro:if value="${mirror_dae == True}">
-                        <mesh filename="package://go2_description/meshes/upperleg.dae" scale="1 1 1"/>
+                        <mesh filename="package://go2_description/meshes/upperleg.stl" scale="1 1 1"/>
                     </xacro:if>
                     <xacro:if value="${mirror_dae == False}">
-                        <mesh filename="package://go2_description/meshes/upperleg_mirror.dae" scale="1 1 1"/>
+                        <mesh filename="package://go2_description/meshes/upperleg_mirror.stl" scale="1 1 1"/>
                     </xacro:if>
                 </geometry>
@@ -111,5 +111,5 @@
                 <origin rpy="0 0 0" xyz="0 0 0"/>
                 <geometry>
-                    <mesh filename="package://go2_description/meshes/lowerleg.dae" scale="1 1 1"/>
+                    <mesh filename="package://go2_description/meshes/lowerleg.stl" scale="1 1 1"/>
                 </geometry>
                 <!-- <material name="orange"/> -->
